File: build/DAISY_DRUM_MACHINE/DAISY_DRUM_MACHINE.kicad_sch (KiCad schematic)
At the start: 70 parts, among them J1 5V, J2 AUDIO_OUT, J3 MIDI_IN, J4 MIDI_IN, U1 TL072, U2 6N138, U3 CD74HC4067M, U4 CD74HC4067M

Commit message: DRM_Mk1
Parts:
- removed D2, D3, D4, D5: BAT85, PCM_Diode_THT_AKL:D_DO-34_SOD68_P7.62mm_Horizontal, symbol PCM_Diode_Schottky_AKL:BAT85
- removed R10, R11: 200k, Resistor_THT:R_Axial_DIN0207_L6.3mm_D2.5mm_P10.16mm_Horizontal, symbol PCM_SL_Resistors:2.2k
- removed R12, R9: 100k, Resistor_THT:R_Axial_DIN0207_L6.3mm_D2.5mm_P10.16mm_Horizontal, symbol PCM_SL_Resistors:2.2k
- removed U1: TL072, PCM_Package_DIP_AKL:DIP-8_W7.62mm_LongPads, symbol PCM_4ms_IC:TL072
