File: build/DAISY_DRUM_MACHINE/DAISY_DRUM_MACHINE.kicad_sch (KiCad schematic)
At the start: 70 parts, among them J1 5V, J2 AUDIO_OUT, J3 MIDI_IN, J4 MIDI_IN, U1 TL072, U2 6N138, U3 CD74HC4067M, U4 CD74HC4067M

Commit message: firmware update
improved midi
Parts:
- removed D2, D3, D4, D5: BAT85, PCM_Diode_THT_AKL:D_DO-34_SOD68_P7.62mm_Horizontal, symbol PCM_Diode_Schottky_AKL:BAT85
- removed R10, R11: 200k, Resistor_THT:R_Axial_DIN0207_L6.3mm_D2.5mm_P10.16mm_Horizontal, symbol PCM_SL_Resistors:2.2k
- removed R12, R9: 100k, Resistor_THT:R_Axial_DIN0207_L6.3mm_D2.5mm_P10.16mm_Horizontal, symbol PCM_SL_Resistors:2.2k
- removed U1: TL072, PCM_Package_DIP_AKL:DIP-8_W7.62mm_LongPads, symbol PCM_4ms_IC:TL072
- R6: value 220R -> 10k

Commit message: updates
Parts:
- C10, C11, C6, C7: footprint Capacitor_THT:C_Disc_D5.0mm_W2.5mm_P2.50mm -> Capacitor_SMD:C_0603_1608Metric_Pad1.08x0.95mm_HandSolder
- J2: footprint PJ307-TRS:PJ307-TRS-SOCKET -> Connector_Audio:Jack_3.5mm_CUI_SJ1-3525N_Horizontal
- R1, R15, R16, R17, R18, R19, R2, R3, R4, R7, R8: footprint Resistor_THT:R_Axial_DIN0207_L6.3mm_D2.5mm_P10.16mm_Horizontal -> Resistor_SMD:R_0603_1608Metric_Pad0.98x0.95mm_HandSolder
- R6: value 10k -> 220R
Changed lines of the file:
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@@
 			)
 		)
-		(property "Footprint" "Resistor_THT:R_Axial_DIN0207_L6.3mm_D2.5mm_P10.16mm_Horizontal"
+		(property "Footprint" "Resistor_SMD:R_0603_1608Metric_Pad0.98x0.95mm_HandSolder"
 			(at 64.008 231.521 0)
 			(effects
@@
 			)
 		)
-		(property "Footprint" "Resistor_THT:R_Axial_DIN0207_L6.3mm_D2.5mm_P10.16mm_Horizontal"
+		(property "Footprint" "Resistor_SMD:R_0603_1608Metric_Pad0.98x0.95mm_HandSolder"
 			(at 64.008 244.221 0)
 			(effects
@@
 			)
 		)
-		(property "Footprint" "Capacitor_THT:C_Disc_D5.0mm_W2.5mm_P2.50mm"
+		(property "Footprint" "Capacitor_SMD:C_0603_1608Metric_Pad1.08x0.95mm_HandSolder"
 			(at 140.97 106.68 0)
 			(effects
@@
 			)
 		)
-		(property "Footprint" "Resistor_THT:R_Axial_DIN0207_L6.3mm_D2.5mm_P10.16mm_Horizontal"
+		(property "Footprint" "Resistor_SMD:R_0603_1608Metric_Pad0.98x0.95mm_HandSolder"
 			(at 42.799 231.648 0)
 			(effects
@@
 			)
 		)
-		(property "Footprint" "Capacitor_THT:C_Disc_D5.0mm_W2.5mm_P2.50mm"
+		(property "Footprint" "Capacitor_SMD:C_0603_1608Metric_Pad1.08x0.95mm_HandSolder"
 			(at 50.8 231.14 0)
 			(effects
@@
 			)
 		)
-		(property "Footprint" "Capacitor_THT:C_Disc_D5.0mm_W2.5mm_P2.50mm"
+		(property "Footprint" "Capacitor_SMD:C_0603_1608Metric_Pad1.08x0.95mm_HandSolder"
 			(at 50.8 243.84 0)
 			(effects
@@
 			)
 		)
-		(property "Footprint" "Resistor_THT:R_Axial_DIN0207_L6.3mm_D2.5mm_P10.16mm_Horizontal"
+		(property "Footprint" "Resistor_SMD:R_0603_1608Metric_Pad0.98x0.95mm_HandSolder"
 			(at 42.799 244.348 0)
 			(effects
@@
 			)
 		)
-		(property "Footprint" "Resistor_THT:R_Axial_DIN0207_L6.3mm_D2.5mm_P10.16mm_Horizontal"
+		(property "Footprint" "Resistor_SMD:R_0603_1608Metric_Pad0.98x0.95mm_HandSolder"
 			(at 132.842 197.739 0)
 			(effects
@@
 			)
 		)
-		(property "Footprint" "PJ307-TRS:PJ307-TRS-SOCKET"
+		(property "Footprint" "Connector_Audio:Jack_3.5mm_CUI_SJ1-3525N_Horizontal"
 			(at 78.74 229.87 0)
 			(effects
@@
 			)
 		)
-		(property "Footprint" "Resistor_THT:R_Axial_DIN0207_L6.3mm_D2.5mm_P10.16mm_Horizontal"
+		(property "Footprint" "Resistor_SMD:R_0603_1608Metric_Pad0.98x0.95mm_HandSolder"
 			(at 123.952 197.739 0)
 			(effects
@@
 			)
 		)
-		(property "Footprint" "Resistor_THT:R_Axial_DIN0207_L6.3mm_D2.5mm_P10.16mm_Horizontal"
+		(property "Footprint" "Resistor_SMD:R_0603_1608Metric_Pad0.98x0.95mm_HandSolder"
 			(at 155.702 197.739 0)
 			(effects
@@
 			)
 		)
-		(property "Footprint" "Capacitor_THT:C_Disc_D5.0mm_W2.5mm_P2.50mm"
+		(property "Footprint" "Capacitor_SMD:C_0603_1608Metric_Pad1.08x0.95mm_HandSolder"
 			(at 140.97 36.83 0)
 			(effects
@@
 			)
 		)
-		(property "Value" "10k"
+		(property "Value" "220R"
 			(at 87.63 175.2599 90)
 			(effects
@@
 			)
 		)
-		(property "Footprint" "Resistor_THT:R_Axial_DIN0207_L6.3mm_D2.5mm_P10.16mm_Horizontal"
+		(property "Footprint" "Resistor_SMD:R_0603_1608Metric_Pad0.98x0.95mm_HandSolder"
 			(at 131.572 152.019 0)
 			(effects
@@
 			)
 		)
-		(property "Footprint" "Resistor_THT:R_Axial_DIN0207_L6.3mm_D2.5mm_P10.16mm_Horizontal"
+		(property "Footprint" "Resistor_SMD:R_0603_1608Metric_Pad0.98x0.95mm_HandSolder"
 			(at 148.082 197.739 0)
 			(effects
@@
 			)
 		)
-		(property "Footprint" "Resistor_THT:R_Axial_DIN0207_L6.3mm_D2.5mm_P10.16mm_Horizontal"
+		(property "Footprint" "Resistor_SMD:R_0603_1608Metric_Pad0.98x0.95mm_HandSolder"
 			(at 140.462 197.739 0)
 			(effects
@@
 			)
 		)
-		(property "Footprint" "Resistor_THT:R_Axial_DIN0207_L6.3mm_D2.5mm_P10.16mm_Horizontal"
+		(property "Footprint" "Resistor_SMD:R_0603_1608Metric_Pad0.98x0.95mm_HandSolder"
 			(at 131.572 82.169 0)
 			(effects

Commit message: Schematic & PCB update
Added drum voice inputs with circuit protection
Parts:
- added C2, C3, C4: 100nF_Ceramic, Capacitor_SMD:C_0603_1608Metric_Pad1.08x0.95mm_HandSolder, symbol PCM_SL_Capacitors:100nF_Ceramic
- added D11, D12, D13, D14, D15, D16, D2, D3, D4, D5: BAT43, PCM_Diode_THT_AKL:D_DO-35_SOD27_P7.62mm_Horizontal, symbol PCM_Diode_Schottky_AKL:BAT43
- added J5: KICK_TRIG_INPUT, Connector_Audio:Jack_3.5mm_CUI_SJ1-3525N_Horizontal, symbol Connector_Audio:AudioJack2_SwitchT
- added J6: SNARE_TRIG_INPUT, Connector_Audio:Jack_3.5mm_CUI_SJ1-3525N_Horizontal, symbol Connector_Audio:AudioJack2_SwitchT
- added J7: HATS_TRIG_INPUT, Connector_Audio:Jack_3.5mm_CUI_SJ1-3525N_Horizontal, symbol Connector_Audio:AudioJack2_SwitchT
- added J8: FM1_TRIG_INPUT, Connector_Audio:Jack_3.5mm_CUI_SJ1-3525N_Horizontal, symbol Connector_Audio:AudioJack2_SwitchT
- added J9: FM2_TRIG_INPUT, Connector_Audio:Jack_3.5mm_CUI_SJ1-3525N_Horizontal, symbol Connector_Audio:AudioJack2_SwitchT
- added R10, R22, R27, R29, R34, R36: 10k, Resistor_SMD:R_0603_1608Metric_Pad0.98x0.95mm_HandSolder, symbol PCM_SL_Resistors:2.2k
- added R11, R12, R20, R23, R24, R25, R30, R31, R32, R35: 100k, Resistor_SMD:R_0603_1608Metric_Pad0.98x0.95mm_HandSolder, symbol PCM_SL_Resistors:2.2k
- added R21, R26, R28, R33, R9: 3.3k, Resistor_SMD:R_0603_1608Metric_Pad0.98x0.95mm_HandSolder, symbol PCM_SL_Resistors:2.2k
- added U1, U5, U6: MCP602, PCM_Package_SO_AKL:SOIC-8_3.9x4.9mm_P1.27mm, symbol Amplifier_Operational:MCP602
- D1: footprint PCM_Diode_THT_AKL:D_DO-35_SOD27_P7.62mm_Horizontal -> Diode_SMD:D_0603_1608Metric_Pad1.05x0.95mm_HandSolder
- J3, J4: footprint PJ307-TRS:PJ307-TRS-SOCKET -> Connector_Audio:Jack_3.5mm_CUI_SJ1-3525N_Horizontal
- R13, R14, R5, R6: footprint Resistor_THT:R_Axial_DIN0207_L6.3mm_D2.5mm_P10.16mm_Horizontal -> Resistor_SMD:R_0603_1608Metric_Pad0.98x0.95mm_HandSolder
Connections:
- net 5V: no longer R14.1
- net A3V3: now also C2.2, C3.2, C4.2, D11.2 (A), D13.2 (A), D15.2 (A), D2.2 (A), D4.2 (A), R21.1, R26.1, R28.1, R33.1, R9.1, U1.8 (V+), U5.8 (V+), U6.8 (V+)
- net AGND: now also C2.1, C3.1, C4.1, D12.1 (K), D14.1 (K), D16.1 (K), D3.1 (K), D5.1 (K), J5.S, J5.TN, J6.S, J6.TN, J7.S, J7.TN, J8.S, J8.TN, J9.S, J9.TN, R10.2, R12.1, R22.2, R23.1, R27.2, R29.2, R30.1, R31.1, R34.2, R35.1, U1.4 (V-), U5.4 (V-), U6.4 (V-)
- net D3V3: now also R14.1, R36.1
- net MIDI_IN: now also R36.2
- net SNARE_TRIG_INPUT: now reaches A1.10 (SPI1_POCI)
- net SNARE_TRIG_INPUT: now also U1.7
- net HATS_TRIG_INPUT: now reaches A1.11 (SPI1_PICO)
- net HATS_TRIG_INPUT: now also U5.1
- net FM1_TRIG_INPUT: now reaches A1.12 (I2C1_SCL)
- net FM1_TRIG_INPUT: now also U5.7
- net FM2_TRIG_INPUT: now reaches A1.13 (I2C1_SDA)
- net FM2_TRIG_INPUT: now also U6.1
- net KICK_TRIG_INPUT: now reaches A1.9 (SPI1_SCK)
- net KICK_TRIG_INPUT: now also U1.1
- new net: D4.1 (K), D5.2 (A), R20.2, R23.2, U1.5 (+)
- new net: D2.1 (K), D3.2 (A), R11.2, R12.2, U1.3 (+)
- new net: R28.2, R29.1, U5.6 (-)
- new net: D15.1 (K), D16.2 (A), R32.2, R35.2, U6.3 (+)
- new net: J7.T, R24.1
- new net: D11.1 (K), D12.2 (A), R24.2, R30.2, U5.3 (+)
- new net: J9.T, R32.1
- new net: R33.2, R34.1, U6.2 (-)
- new net: J5.T, R11.1
- new net: R26.2, R27.1, U5.2 (-)
- new net: R21.2, R22.1, U1.6 (-)
- new net: D13.1 (K), D14.2 (A), R25.2, R31.2, U5.5 (+)
- new net: R10.1, R9.2, U1.2 (-)
- new net: J8.T, R25.1
- new net: J6.T, R20.1
- no-connect marks 3 -> 6
Other:
- note added: "INPUT TRIGGERS"
- note added: "LED Triggers"
- note added: "MUX1"
- note added: "MUX2"
- note added: "POTS"
- note added: "SEED"
- moved on the sheet: A1, C1, C10, C11, C6, C7, C8, C9, D10, D6, D7, D8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
