File: build/DAISY_DRUM_MACHINE/DAISY_DRUM_MACHINE.kicad_pcb (KiCad board)
At the start: 2 copper layers, 312.2 x 242 mm, 122 parts, among them J1 5V, J2 AUDIO_OUT, J3 MIDI_IN, J4 MIDI_IN, U2 6N138, U3 CD74HC4067M, U4 CD74HC4067M

Commit message: updates
Parts:
- C10, C11, C6, C7: footprint Capacitor_THT:C_Disc_D5.0mm_W2.5mm_P2.50mm -> Capacitor_SMD:C_0603_1608Metric_Pad1.08x0.95mm_HandSolder
- J2: footprint PJ307-TRS:PJ307-TRS-SOCKET -> Connector_Audio:Jack_3.5mm_CUI_SJ1-3525N_Horizontal
- R1, R15, R16, R17, R18, R19, R2, R3, R4, R7, R8: footprint Resistor_THT:R_Axial_DIN0207_L6.3mm_D2.5mm_P10.16mm_Horizontal -> Resistor_SMD:R_0603_1608Metric_Pad0.98x0.95mm_HandSolder
- moved C7 33.8 mm to (39.0, 94.0), turned to 90 degrees
- moved C6 32.0 mm to (39.0, 89.6)
- moved C9 30.5 mm to (34.2, 93.0), turned to 180 degrees
- moved C8 25.5 mm to (34.5, 88.0), turned to 180 degrees
- moved R4 20.6 mm to (30.0, 92.1), turned to -90 degrees
- moved R2 17.6 mm to (42.0, 93.0), turned to 180 degrees
- moved R1 17.3 mm to (42.0, 90.5), turned to 180 degrees
- moved R3 11.2 mm to (30.5, 87.0), turned to -90 degrees
- moved R19 9.00 mm to (315.0, 79.0)
- moved C10 4.27 mm to (91.5, 102.5), turned to 0 degrees
- moved C11 2.75 mm to (95.5, 123.6), turned to 90 degrees
- moved R15 2.34 mm to (168.6, 79.2)
- moved R7 1.08 mm to (98.5, 135.5)
Connections:
- D10 pad 1: unconnected-(D10-Pad1) -> Net-(D10-Pad1)
- R19 pad 1: unconnected-(R19-Pad1) -> Net-(D10-Pad1)
Routing:
- net R_OUT: track 41.1 -> 5.66 mm
- net Net-(C9-Pad2): track 21.9 -> 42.8 mm
- net L_OUT: track 22.1 -> 5.88 mm
- net Net-(C8-Pad2): track 21.9 -> 36.2 mm
- net Net-(D10-Pad1): track 0.00 -> 11.4 mm, vias 0 -> 1
- net AGND: track 17.2 -> 6.96 mm, vias 2 -> 3
- net GND: track 366.9 -> 374.9 mm, vias 2 -> 8
- net unconnected-(R19-Pad1): track 3.00 -> 0.00 mm
- net A3V3: track 798.7 -> 800.8 mm, vias 2 -> 3
- net Net-(C7-Pad2): track 8.54 -> 6.98 mm
- net Net-(D6-Pad1): track 3.47 -> 4.90 mm, vias 0 -> 1
- net Net-(U3-~{E}): track 4.79 -> 3.88 mm
- net Net-(C6-Pad2): track 8.33 -> 7.63 mm

Commit message: pcb updates
Parts:
- removed the G*** at (42.8, 176.8)
- removed the G*** at (43.0, 186.0)
- removed the REF** at (23.8, 170.5)
- added REF**: MountingHole_3.2mm_M3, MountingHole:MountingHole_3.2mm_M3, F.Cu at (23.8, 192.0)
- added REF**: MountingHole_3.2mm_M3, MountingHole:MountingHole_3.2mm_M3, F.Cu at (23.8, 71.0)
- moved R14 121.5 mm to (121.8, 191.6)
- moved A1 121.5 mm to (48.8, 168.9)
- moved C1 121.5 mm to (83.5, 185.5)
- moved C10 121.5 mm to (91.5, 224.0)
- moved C7 121.5 mm to (39.0, 215.5)
- moved C8 121.5 mm to (34.5, 209.5)
- moved C9 121.5 mm to (34.2, 214.5)
- moved D1 121.5 mm to (95.0, 184.3)
- moved D10 121.5 mm to (302.8, 200.8)
- moved D6 121.5 mm to (162.8, 200.8)
- moved D7 121.5 mm to (197.8, 200.8)
- moved D8 121.5 mm to (222.8, 200.8)
- moved D9 121.5 mm to (257.8, 200.8)
- moved G*** 121.5 mm to (237.0, 234.8)
- moved J1 121.5 mm to (83.0, 180.5)
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Other:
- outline, holes or cut-outs redrawn
