File: build/DAISY_DRUM_MACHINE/DAISY_DRUM_MACHINE.kicad_pcb (KiCad board)
At the start: 2 copper layers, 312.2 x 242 mm, 121 parts, among them J1 5V, J2 AUDIO_OUT, J3 MIDI_IN, J4 MIDI_IN, U2 6N138, U3 CD74HC4067M, U4 CD74HC4067M

Commit message: Schematic & PCB update
Added drum voice inputs with circuit protection
Parts:
- removed the REF** at (133.8, 282.0)
- removed the REF** at (133.8, 171.0)
- removed the REF** at (133.8, 161.0)
- removed the REF** at (133.8, 50.0)
- added C2: 100nF_Ceramic, Capacitor_SMD:C_0603_1608Metric_Pad1.08x0.95mm_HandSolder, F.Cu at (142.8, 78.5)
- added C3: 100nF_Ceramic, Capacitor_SMD:C_0603_1608Metric_Pad1.08x0.95mm_HandSolder, F.Cu at (240.9, 72.0)
- added C4: 100nF_Ceramic, Capacitor_SMD:C_0603_1608Metric_Pad1.08x0.95mm_HandSolder, F.Cu at (281.2, 66.5)
- added D11: BAT43, PCM_Diode_THT_AKL:D_DO-35_SOD27_P7.62mm_Horizontal, F.Cu at (213.2, 50.3)
- added D12: BAT43, PCM_Diode_THT_AKL:D_DO-35_SOD27_P7.62mm_Horizontal, F.Cu at (205.6, 53.0)
- added D13: BAT43, PCM_Diode_THT_AKL:D_DO-35_SOD27_P7.62mm_Horizontal, F.Cu at (247.2, 49.7)
- added D14: BAT43, PCM_Diode_THT_AKL:D_DO-35_SOD27_P7.62mm_Horizontal, F.Cu at (239.6, 52.3)
- added D15: BAT43, PCM_Diode_THT_AKL:D_DO-35_SOD27_P7.62mm_Horizontal, F.Cu at (292.3, 49.4)
- added D16: BAT43, PCM_Diode_THT_AKL:D_DO-35_SOD27_P7.62mm_Horizontal, F.Cu at (284.7, 52.1)
- added D2: BAT43, PCM_Diode_THT_AKL:D_DO-35_SOD27_P7.62mm_Horizontal, F.Cu at (153.8, 49.5)
- added D3: BAT43, PCM_Diode_THT_AKL:D_DO-35_SOD27_P7.62mm_Horizontal, F.Cu at (146.2, 52.2)
- added D4: BAT43, PCM_Diode_THT_AKL:D_DO-35_SOD27_P7.62mm_Horizontal, F.Cu at (187.2, 49.5)
- added D5: BAT43, PCM_Diode_THT_AKL:D_DO-35_SOD27_P7.62mm_Horizontal, F.Cu at (179.7, 52.1)
- added J5: KICK_TRIG_INPUT, Connector_Audio:Jack_3.5mm_CUI_SJ1-3525N_Horizontal, F.Cu at (161.5, 49.5)
- added J6: SNARE_TRIG_INPUT, Connector_Audio:Jack_3.5mm_CUI_SJ1-3525N_Horizontal, F.Cu at (196.5, 49.5)
- added J7: HATS_TRIG_INPUT, Connector_Audio:Jack_3.5mm_CUI_SJ1-3525N_Horizontal, F.Cu at (221.5, 49.5)
- added J8: FM1_TRIG_INPUT, Connector_Audio:Jack_3.5mm_CUI_SJ1-3525N_Horizontal, F.Cu at (256.5, 49.5)
- added J9: FM2_TRIG_INPUT, Connector_Audio:Jack_3.5mm_CUI_SJ1-3525N_Horizontal, F.Cu at (301.5, 49.5)
- added R10: 10k, Resistor_SMD:R_0603_1608Metric_Pad0.98x0.95mm_HandSolder, F.Cu at (141.8, 65.5)
- added R11: 100k, Resistor_SMD:R_0603_1608Metric_Pad0.98x0.95mm_HandSolder, F.Cu at (153.3, 54.5)
- added R12: 100k, Resistor_SMD:R_0603_1608Metric_Pad0.98x0.95mm_HandSolder, F.Cu at (139.1, 68.0)
- added R20: 100k, Resistor_SMD:R_0603_1608Metric_Pad0.98x0.95mm_HandSolder, F.Cu at (188.5, 54.5)
- added R21: 3.3k, Resistor_SMD:R_0603_1608Metric_Pad0.98x0.95mm_HandSolder, F.Cu at (145.2, 78.5)
- added R22: 10k, Resistor_SMD:R_0603_1608Metric_Pad0.98x0.95mm_HandSolder, F.Cu at (147.0, 80.3)
- added R23: 100k, Resistor_SMD:R_0603_1608Metric_Pad0.98x0.95mm_HandSolder, F.Cu at (137.0, 76.2)
- added R24: 100k, Resistor_SMD:R_0603_1608Metric_Pad0.98x0.95mm_HandSolder, F.Cu at (213.5, 55.4)
- added R25: 100k, Resistor_SMD:R_0603_1608Metric_Pad0.98x0.95mm_HandSolder, F.Cu at (248.2, 54.5)
- added R26: 3.3k, Resistor_SMD:R_0603_1608Metric_Pad0.98x0.95mm_HandSolder, F.Cu at (231.5, 73.5)
- added R27: 10k, Resistor_SMD:R_0603_1608Metric_Pad0.98x0.95mm_HandSolder, F.Cu at (229.9, 75.5)
- added R28: 3.3k, Resistor_SMD:R_0603_1608Metric_Pad0.98x0.95mm_HandSolder, F.Cu at (240.9, 75.4)
- added R29: 10k, Resistor_SMD:R_0603_1608Metric_Pad0.98x0.95mm_HandSolder, F.Cu at (242.6, 77.4)
- added R30: 100k, Resistor_SMD:R_0603_1608Metric_Pad0.98x0.95mm_HandSolder, F.Cu at (231.4, 77.1)
- added R31: 100k, Resistor_SMD:R_0603_1608Metric_Pad0.98x0.95mm_HandSolder, F.Cu at (238.8, 79.7)
- added R32: 100k, Resistor_SMD:R_0603_1608Metric_Pad0.98x0.95mm_HandSolder, F.Cu at (293.3, 54.4)
- added R33: 3.3k, Resistor_SMD:R_0603_1608Metric_Pad0.98x0.95mm_HandSolder, F.Cu at (279.9, 59.5)
- added R34: 10k, Resistor_SMD:R_0603_1608Metric_Pad0.98x0.95mm_HandSolder, F.Cu at (276.4, 59.4)
- added R35: 100k, Resistor_SMD:R_0603_1608Metric_Pad0.98x0.95mm_HandSolder, F.Cu at (282.2, 64.0)
- added R36: 10k, Resistor_SMD:R_0603_1608Metric_Pad0.98x0.95mm_HandSolder, F.Cu at (94.2, 79.0)
- added R9: 3.3k, Resistor_SMD:R_0603_1608Metric_Pad0.98x0.95mm_HandSolder, F.Cu at (142.8, 68.2)
- added REF**: MountingHole_3.2mm_M3, MountingHole:MountingHole_3.2mm_M3, F.Cu at (72.0, 50.2)
- added REF**: MountingHole_3.2mm_M3, MountingHole:MountingHole_3.2mm_M3, F.Cu at (72.0, 171.2)
- added U1: MCP602, PCM_Package_SO_AKL:SOIC-8_3.9x4.9mm_P1.27mm, F.Cu at (140.8, 73.0)
- added U5: MCP602, PCM_Package_SO_AKL:SOIC-8_3.9x4.9mm_P1.27mm, F.Cu at (236.2, 75.0)
- added U6: MCP602, PCM_Package_SO_AKL:SOIC-8_3.9x4.9mm_P1.27mm, F.Cu at (277.3, 64.7)
- D1: footprint PCM_Diode_THT_AKL:D_DO-35_SOD27_P7.62mm_Horizontal -> Diode_SMD:D_0603_1608Metric_Pad1.05x0.95mm_HandSolder
- J3, J4: footprint PJ307-TRS:PJ307-TRS-SOCKET -> Connector_Audio:Jack_3.5mm_CUI_SJ1-3525N_Horizontal
- R13, R14, R5, R6: footprint Resistor_THT:R_Axial_DIN0207_L6.3mm_D2.5mm_P10.16mm_Horizontal -> Resistor_SMD:R_0603_1608Metric_Pad0.98x0.95mm_HandSolder
- moved R14 131.2 mm to (119.7, 60.4), turned to 0 degrees
- moved REF** 129.5 mm to (171.2, 160.5)
- moved REF** 129.5 mm to (171.2, 49.5)
- moved REF** 128.5 mm to (171.2, 170.5)
- moved REF** 128.5 mm to (171.2, 281.5)
- moved D1 127.7 mm to (94.9, 56.6)
- moved R5 123.5 mm to (97.0, 61.0), turned to 90 degrees
- moved R6 121.5 mm to (94.2, 77.2)
- moved G*** 121.0 mm to (169.8, 231.0)
- moved G*** 121.0 mm to (117.8, 209.1)
- moved A1 121.0 mm to (48.8, 47.9)
- moved C1 121.0 mm to (83.5, 64.5)
- moved C10 121.0 mm to (91.5, 103.0)
- moved C7 121.0 mm to (39.0, 94.5)
- moved C8 121.0 mm to (34.5, 88.5)
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Connections:
- A1 pad 10: unconnected-(A1-SPI1_POCI-Pad10) -> SNARE_TRIG_INPUT
- A1 pad 11: unconnected-(A1-SPI1_PICO-Pad11) -> HATS_TRIG_INPUT
- A1 pad 12: unconnected-(A1-I2C1_SCL-Pad12) -> FM1_TRIG_INPUT
- A1 pad 13: unconnected-(A1-I2C1_SDA-Pad13) -> FM2_TRIG_INPUT
- A1 pad 9: unconnected-(A1-SPI1_SCK-Pad9) -> KICK_TRIG_INPUT
- R14 pad 1: 5V -> D3V3
Routing:
- net FM2_TRIG_INPUT: track 0.00 -> 424.7 mm, vias 0 -> 3
- net HATS_TRIG_INPUT: track 0.00 -> 393.0 mm, vias 0 -> 3
- net FM1_TRIG_INPUT: track 0.00 -> 385.9 mm, vias 0 -> 3
- net A3V3: track 800.8 -> 1148.6 mm, vias 3 -> 4
- net KICK_TRIG_INPUT: track 0.00 -> 316.8 mm, vias 0 -> 3
- net SNARE_TRIG_INPUT: track 0.00 -> 294.0 mm, vias 0 -> 5
- net Net-(D13-K): track 0.00 -> 77.8 mm
- net Net-(D4-K): track 0.00 -> 76.1 mm, vias 0 -> 1
- net AGND: track 6.96 -> 62.7 mm, vias 3 -> 12
- net 5V: track 84.7 -> 31.2 mm
- net Net-(D11-K): track 0.00 -> 52.7 mm, vias 0 -> 4
- net D3V3: track 49.9 -> 84.2 mm
- net Net-(D2-K): track 0.00 -> 29.8 mm, vias 0 -> 2
- net Net-(D15-K): track 0.00 -> 27.3 mm
- net Net-(U1B--): track 0.00 -> 12.1 mm
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Other:
- outline, holes or cut-outs redrawn
